File: ruche.kicad_pcb (KiCad board)
At the start: 2 copper layers, 92.8 x 99.9 mm, 190 parts, among them IC1 CN3791, IC2 MAX17048G+, IC3 L86-M33, IC4 SHT41-AD1B-R3, IC5 HX711, IC6 HX711, IC7 HX711, IC8 HX711, IC9 FS312F-G, J1 Conn_01x02, J10 Conn_01x04, J11 Conn_01x04, J12 Conn_01x04, J13 Micro_SD_Card, J14 Conn_01x03, J15 Conn_01x04, J16 Conn_01x04, J17 Conn_01x04, J18 Conn_01x04, J19 Conn_01x02, J2 Conn_01x04, J20 USB_C_Receptacle_USB2.0 USB41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, J3 Conn_01x03, J4 Conn_01x03, J5 Conn_01x04, J6 Conn_01x02, J7 Conn_01x02, J8 Conn_01x03, J9 Conn_01x03, Q1 AO3401A, Q2 MMBT4403, Q3 MMBT4403, Q4 MMBT4403, Q5 MMBT4403, Q6 UMH3N, Q7 DMG2301L, Q8 FS8205, SW1 SW_Push, U1 CP2102N-A02-GQFN24, U2 MS5611-01BA, U3 XC6220B331MR, U4 TCA9548APWR, U5 XC6220B331MR, U6 ESP32-S3-WROOM-2, U7 1043, U9 XC6220B331MR

Commit message: Update
Parts:
- added R42: 499/5%, Resistor_SMD:R_0603_1608Metric, F.Cu at (151.1, 109.5)
- U6: value ESP32-S3-WROOM-2 -> Heltec_Wireless_shell_V3; footprint Espressif:ESP32-S3-WROOM-1U -> Empreintes:Heltec Wireless shell V3
- moved S1 36.1 mm to (117.7, 116.3), turned to -90 degrees
- moved G*** 12.8 mm to (125.2, 117.9)
- moved U6 8.58 mm to (132.1, 109.7), turned to 180 degrees
Connections:
- U6 pad 1: GND -> unconnected-(U6-Pad1)
- U6 pad 10: unconnected-(U6-Pad10) -> DAT1
- U6 pad 11: unconnected-(U6-Pad11) -> SDO-MISO-D10
- U6 pad 12: unconnected-(U6-Pad12) -> CMD-MOSI-D8
- U6 pad 13: unconnected-(U6-Pad13) -> CLK-SCK-D9
- U6 pad 14: Start_modules -> SD3-CS-D7
- U6 pad 15: Tilt_led_alarm -> UORXD
- U6 pad 16: unconnected-(U6-Pad16) -> Net-(R42-Pad1)
- U6 pad 17: TX_GPS -> RX_GPS
- U6 pad 18: RX_GPS -> TX_GPS
- U6 pad 19: Start_GPS -> unconnected-(U6-Pad19)
- U6 pad 2: +3V3 -> unconnected-(U6-Pad2)
- U6 pad 21: unconnected-(U6-Pad21) -> INT1
- U6 pad 22: INT1 -> unconnected-(U6-Pad22)
- U6 pad 23: DS18b20 -> EN
- U6 pad 24: unconnected-(U6-Pad24) -> DS18b20
- U6 pad 25: unconnected-(U6-Pad25) -> DAT2
- U6 pad 27: IO0 -> unconnected-(U6-Pad27)
- U6 pad 28: SD3-CS-D7 -> CLK1
- U6 pad 29: CMD-MOSI-D8 -> CLK2
- U6 pad 3: EN -> Net-(U6-Pad3)
- U6 pad 30: DAT4 -> unconnected-(U6-Pad30)
- U6 pad 31: CLK4 -> CLK3
- U6 pad 33: CLK3 -> unconnected-(U6-Pad33)
- U6 pad 34: DAT2 -> IO0
- U6 pad 35: CLK2 -> SDA
- U6 pad 36: UORXD -> SCL
- U6 pad 37: UOTXD -> unconnected-(U6-Pad37)
- U6 pad 38: DAT1 -> unconnected-(U6-Pad38)
- U6 pad 39: CLK1 -> unconnected-(U6-Pad39)
- U6 pad 4: SDO-MISO-D10 -> Net-(U6-Pad3)
- U6 pad 40: GND -> unconnected-(U6-Pad40)
- U6 pad 5: CLK-SCK-D9 -> CLK4
- U6 pad 6: SDA -> DAT4
- U6 pad 7: SCL -> Tilt_led_alarm
- U6 pad 8: unconnected-(U6-Pad8) -> Start_GPS
- U6 pad 9: unconnected-(U6-Pad9) -> Start_modules
Routing:
- net INT1: track 42.2 -> 0.00 mm, vias 1 -> 0
- net SDO-MISO-D10: track 29.4 -> 0.00 mm, vias 2 -> 0
- net CLK-SCK-D9: track 34.5 -> 63.9 mm, vias 2 -> 4
- net DAT4: track 21.5 -> 0.00 mm
- net CLK4: track 21.3 -> 0.00 mm
- net CLK1: track 19.5 -> 0.00 mm
- net DAT1: track 19.1 -> 0.00 mm
- net VCC: track 398.7 -> 381.1 mm
- net unconnected-(U6-Pad8): track 16.9 -> 0.00 mm, vias 1 -> 0
- net DS18b20: track 108.2 -> 93.3 mm
- net DAT3: track 10.6 -> 0.00 mm
- net CLK3: track 10.5 -> 0.00 mm
- net DAT2: track 9.58 -> 0.00 mm
- net EN: track 88.2 -> 80.3 mm
- net CLK2: track 9.76 -> 16.9 mm, vias 0 -> 1
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
Commit message: Update
Parts:
- moved C57 26.0 mm to (151.7, 88.3)
- moved C59 23.9 mm to (150.4, 94.6)
- moved R48 23.9 mm to (150.4, 91.6)
- moved C58 23.1 mm to (150.1, 88.5)
- moved R10 14.3 mm to (129.1, 111.4)
- moved R42 1.05 mm to (151.0, 108.5)
- moved J19 0.17 mm to (143.3, 122.3)
Connections:
- U6 pad 10: DAT1 -> unconnected-(U6-Pad10)
- U6 pad 20: unconnected-(U6-Pad20) -> CLK4
- U6 pad 21: INT1 -> DAT4
- U6 pad 24: DS18b20 -> DAT3
- U6 pad 25: DAT2 -> CLK3
- U6 pad 26: unconnected-(U6-Pad26) -> Start_GPS
- U6 pad 27: unconnected-(U6-Pad27) -> INT1
- U6 pad 28: CLK1 -> Start_modules
- U6 pad 29: CLK2 -> unconnected-(U6-Pad29)
- U6 pad 3: Net-(U6-Pad3) -> +3V3
- U6 pad 31: CLK3 -> unconnected-(U6-Pad31)
- U6 pad 32: DAT3 -> unconnected-(U6-Pad32)
- U6 pad 33: unconnected-(U6-Pad33) -> DS18b20
- U6 pad 4: Net-(U6-Pad3) -> +3V3
- U6 pad 5: CLK4 -> DAT1
- U6 pad 6: DAT4 -> CLK1
- U6 pad 7: Tilt_led_alarm -> CLK2
- U6 pad 8: Start_GPS -> unconnected-(U6-Pad8)
- U6 pad 9: Start_modules -> DAT2
Routing:
- net +3V3: track 145.6 -> 183.7 mm
- net SDO-MISO-D10: track 0.00 -> 37.1 mm, vias 0 -> 2
- net IO0: track 36.4 -> 64.9 mm, vias 0 -> 2
- net CLK-SCK-D9: track 63.9 -> 41.7 mm, vias 4 -> 2
- net CLK1: track 0.00 -> 22.1 mm
- net DAT1: track 0.00 -> 20.6 mm
- net DAT4: track 0.00 -> 19.0 mm
- net CLK3: track 0.00 -> 18.9 mm
- net RX_GPS: track 44.4 -> 62.9 mm
- net VCC: track 381.1 -> 399.0 mm
- net DAT3: track 0.00 -> 17.7 mm
- net DS18b20: track 93.3 -> 75.7 mm
- net CLK4: track 0.00 -> 17.2 mm
- net TX_GPS: track 41.6 -> 57.6 mm
- net INT1: track 0.00 -> 15.4 mm
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
Commit message: Update
Parts:
- added J21: Conn_01x02, Connector_JST:JST_PH_B2B-PH-K_1x02_P2.00mm_Vertical, F.Cu at (168.3, 72.1)
- added R43: 100k, Resistor_SMD:R_0603_1608Metric, F.Cu at (129.4, 107.8)
- moved D7 25.5 mm to (151.0, 105.2)
- moved R11 25.3 mm to (151.0, 102.4)
- moved FID2 7.22 mm to (175.1, 79.0)
Connections:
- U6 pad 10: unconnected-(U6-Pad10) -> DAT1
- U6 pad 22: unconnected-(U6-Pad22) -> CLK1
- U6 pad 31: unconnected-(U6-Pad31) -> Rain_gauge
- U6 pad 5: DAT1 -> unconnected-(U6-Pad5)
- U6 pad 6: CLK1 -> unconnected-(U6-Pad6)
- U6 pad 8: unconnected-(U6-Pad8) -> Tilt_led_alarm
Routing:
- net Rain_gauge: track 0.00 -> 63.8 mm, vias 0 -> 2
- net CLK1: track 22.1 -> 49.4 mm, vias 0 -> 2
- net SCL: track 146.1 -> 138.3 mm, vias 9 -> 7
- net DAT1: track 20.6 -> 26.0 mm
- net EN: track 80.4 -> 83.8 mm
- net GND: track 43.7 -> 46.9 mm, vias 285 -> 286
- net +3V3: track 183.7 -> 186.1 mm
- net Tilt_led_alarm: track 3.49 -> 5.38 mm, vias 0 -> 2
- net UOTXD: track 54.6 -> 54.0 mm
Other:
- board text added: "Rain gauge"

Commit message: Update
Parts:
- removed JP1: SolderJumper_3_Open, Jumper:SolderJumper-3_P1.3mm_Open_RoundedPad1.0x1.5mm_NumberLabels
- added C65: 0.1µF, Capacitor_SMD:C_0805_2012Metric, F.Cu at (152.6, 146.7)
- added R54: 10K, Resistor_SMD:R_0603_1608Metric, F.Cu at (151.9, 151.5)
- added SW2: SW_Push, Empreintes:PTS636SL43SMTRLFS, F.Cu at (149.8, 134.5)
- J4: value Conn_01x03 -> Conn_01x02; footprint Connector_JST:JST_PH_B3B-PH-K_1x03_P2.00mm_Vertical -> Connector_JST:JST_PH_B2B-PH-K_1x02_P2.00mm_Vertical
- moved J4 22.4 mm to (153.2, 161.3), turned to -90 degrees
- moved G*** 18.8 mm to (124.1, 99.0)
- moved FID3 10.8 mm to (171.7, 165.1)
- moved SW1 9.72 mm to (159.7, 142.1), turned to 0 degrees
- moved G*** 5.92 mm to (135.8, 129.8)
- moved J21 0.23 mm to (168.5, 72.1)
- moved D11 0.15 mm to (165.6, 154.1)
Connections:
- J4 pad 1: A0/D15 -> VBAT
- J4 pad 2: Net-(J4-Pad2) -> GND
Routing:
- net GND: track 46.9 -> 57.6 mm, vias 286 -> 299
- net +5V: track 68.8 -> 59.4 mm
- net Net-(J4-Pad2): track 8.00 -> 0.00 mm
- net IO0: track 64.6 -> 71.5 mm
- net EN: track 83.8 -> 88.2 mm
- net +3V3: track 186.1 -> 190.0 mm
- net DTR: track 5.01 -> 8.62 mm
- net Rain_gauge: track 63.8 -> 62.9 mm
- net VCC: track 399.0 -> 398.4 mm
Other:
- board text added: "+"
- board text added: "-"
- board text added: "18650 Li-ion battery"
- board text added: "Bat"
- board text added: "Boot"
- board text added: "Opensource connected hive V0.4 by Ratamuse"
- board text added: "P"
- board text added: "R B W G"
- board text added: "Reset PB"
- board text added: "Spare I2C"
- board text removed: "I2C"
- board text removed: "Opensource connected hive V0.2 by Ratamuse"
- board text removed: "R B Y W G"

Commit message: Update
Parts:
- C51, C60: footprint Capacitor_SMD:C_0603_1608Metric -> Capacitor_SMD:C_0805_2012Metric
- C52, C61, C65: footprint Capacitor_SMD:C_0805_2012Metric -> Capacitor_SMD:C_0603_1608Metric
- moved C60 1.65 mm to (158.2, 156.5)
- moved C52 1.63 mm to (137.8, 141.7)
- moved C61 1.62 mm to (156.6, 156.3)
- moved C51 1.59 mm to (139.4, 141.8)
