File: ruche.kicad_pcb (KiCad board)
At the start: 2 copper layers, 92.8 x 99.9 mm, 195 parts, among them IC1 CN3791, IC2 MAX17048G+, IC3 L86-M33, IC4 SHT41-AD1B-R3, IC5 HX711, IC6 HX711, IC7 HX711, IC8 HX711, IC9 FS312F-G, J1 Conn_01x02, J10 Conn_01x04, J11 Conn_01x04, J12 Conn_01x04, J13 Micro_SD_Card, J14 Conn_01x03, J15 Conn_01x04, J16 Conn_01x04, J17 Conn_01x04, J18 Conn_01x04, J19 Conn_01x02, J2 Conn_01x04, J20 USB_C_Receptacle_USB2.0 USB41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, J21 Conn_01x02, J3 Conn_01x03, J4 Conn_01x02, J5 Conn_01x04, J6 Conn_01x02, J7 Conn_01x02, J8 Conn_01x03, J9 Conn_01x03, Q1 AO3401A, Q2 MMBT4403, Q3 MMBT4403, Q4 MMBT4403, Q5 MMBT4403, Q6 UMH3N, Q7 DMG2301L, Q8 FS8205, SW1 SW_Push, SW2 SW_Push, U1 CP2102N-A02-GQFN24, U2 MS5611-01BA, U3 XC6220B331MR, U4 TCA9548APWR, U5 XC6220B331MR, U6 Heltec_Wireless_shell_V3, U7 1043, U9 XC6220B331MR

Commit message: Update
Parts:
- R1: value 2K -> 10K
- moved R48 40.3 mm to (142.2, 131.0), turned to 0 degrees
- moved C59 24.7 mm to (145.6, 118.9), turned to 0 degrees
- moved D7 24.1 mm to (129.9, 93.7), turned to -90 degrees
- moved C57 23.5 mm to (128.2, 90.2), turned to -90 degrees
- moved R11 21.9 mm to (129.9, 96.6), turned to -90 degrees
- moved R43 21.7 mm to (151.1, 107.8)
- moved R42 21.0 mm to (130.1, 109.3), turned to -90 degrees
- moved C58 20.2 mm to (129.9, 88.5)
- moved R10 3.50 mm to (128.3, 114.8), turned to 90 degrees
Connections:
- U6 pad 10: DAT1 -> SDA
- U6 pad 20: CLK4 -> Start_GPS
- U6 pad 22: CLK1 -> CLK4
- U6 pad 24: DAT3 -> CLK3
- U6 pad 25: CLK3 -> DAT3
- U6 pad 26: Start_GPS -> CLK1
- U6 pad 33: DS18b20 -> unconnected-(U6-Pad33)
- U6 pad 35: SDA -> DAT1
- U6 pad 36: SCL -> DAT2
- U6 pad 38: unconnected-(U6-Pad38) -> CLK2
- U6 pad 7: CLK2 -> DS18b20
- U6 pad 9: DAT2 -> SCL
Routing:
- net EN: track 88.2 -> 59.7 mm
- net INT1: track 15.4 -> 32.7 mm, vias 0 -> 2
- net RX_GPS: track 62.9 -> 48.3 mm
- net TX_GPS: track 57.6 -> 43.6 mm
- net IO0: track 71.5 -> 59.6 mm
- net UORXD: track 51.0 -> 62.4 mm
- net UOTXD: track 54.0 -> 64.4 mm, vias 2 -> 4
- net CLK1: track 49.7 -> 40.1 mm
- net Start_modules: track 38.2 -> 47.3 mm
- net CMD-MOSI-D8: track 43.0 -> 36.7 mm
- net SD3-CS-D7: track 45.3 -> 39.2 mm
- net SDO-MISO-D10: track 37.0 -> 31.4 mm
- net CLK3: track 19.4 -> 15.1 mm
- net DAT3: track 17.9 -> 13.8 mm
- net CLK4: track 17.7 -> 21.6 mm
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
Commit message: update
Parts:
- moved D2 2.67 mm to (98.5, 153.9)
Routing:
- net Net-(D1-Pad1): track 27.1 -> 24.4 mm
- net Vsolar: track 48.6 -> 50.9 mm

Commit message: update
Routing:
- net Rain_gauge: track 59.2 -> 58.2 mm
- net Start_GPS: track 19.3 -> 18.3 mm
- net EN: track 59.7 -> 59.2 mm

Commit message: update
Parts:
- moved G*** 4.15 mm to (123.7, 103.2)
- moved R49 1.66 mm to (161.5, 154.3), turned to 180 degrees
- moved D14 0.44 mm to (161.4, 156.0)
Routing:
- net VCC: track 401.7 -> 399.2 mm
- net VBUS: track 25.3 -> 25.9 mm
- net VBAT: track 62.9 -> 63.5 mm, vias 3 -> 4
- net GND: track 54.4 -> 54.2 mm, vias 297 -> 301

Commit message: Revert "update"
This reverts commit 9afc669c055c7e8087787cb6fdf10dddd7845243.
Parts:
- moved G*** 4.15 mm to (124.1, 99.0)
- moved R49 1.66 mm to (163.1, 154.3), turned to 0 degrees
- moved D14 0.44 mm to (161.4, 155.6)
Routing:
- net VCC: track 399.2 -> 401.7 mm
- net VBUS: track 25.9 -> 25.3 mm
- net VBAT: track 63.5 -> 62.9 mm, vias 4 -> 3
- net GND: track 54.2 -> 54.4 mm, vias 301 -> 297
