File: ruche.kicad_sch (KiCad schematic)
At the start: 45 parts, among them IC2 MAX17048G+, IC3 L86-M33, IC4 SHT41-AD1B-R3, J13 Micro_SD_Card, J19 Conn_01x02, U2 MS5611-01BA, U3 XC6220B331MR, U5 XC6220B331MR, U9 XC6220B331MR

Commit message: Update
Parts:
- added J21: Conn_01x02, Connector_JST:JST_PH_B2B-PH-K_1x02_P2.00mm_Vertical, symbol Connector_Generic:Conn_01x02
- added R43: 100k, Resistor_SMD:R_0603_1608Metric, symbol Device:R
Connections:
- net +3V3: now also R43.1
- net GND: now also J21.2 (Pin_2)
- new net Rain_gauge: J21.1 (Pin_1), R43.2
Other:
- note added: "Pluviomètre"
Changed lines of the file:
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@@
   (junction (at 53.34 72.39) (diameter 0) (color 0 0 0 0)
   )
+  (junction (at 156.464 84.074) (diameter 0) (color 0 0 0 0)
+  )
   (junction (at 246.38 95.25) (diameter 0) (color 0 0 0 0)
   )
@@
   (junction (at 113.03 96.52) (diameter 0) (color 0 0 0 0)
   )
+  (wire (pts (xy 156.464 84.074) (xy 156.464 80.264))
+    (stroke (width 0) (type default) (color 0 0 0 0))
+  )
   (wire (pts (xy 135.89 138.43) (xy 135.89 140.97))
     (stroke (width 0) (type default) (color 0 0 0 0))
@@
     (stroke (width 0) (type default) (color 0 0 0 0))
   )
+  (wire (pts (xy 156.464 72.644) (xy 156.464 70.104))
+    (stroke (width 0) (type default) (color 0 0 0 0))
+  )
   (wire (pts (xy 31.75 69.85) (xy 31.75 76.2))
     (stroke (width 0) (type default) (color 0 0 0 0))
@@
     (stroke (width 0) (type default) (color 0 0 0 0))
   )
+  (wire (pts (xy 167.894 84.074) (xy 156.464 84.074))
+    (stroke (width 0) (type default) (color 0 0 0 0))
+  )
   (polyline (pts (xy 123.19 110.49) (xy 123.19 114.3))
     (stroke (width 0) (type default) (color 0 0 0 0))
@@
     (stroke (width 0) (type default) (color 0 0 0 0))
   )
+  (wire (pts (xy 167.894 86.614) (xy 160.274 86.614))
+    (stroke (width 0) (type default) (color 0 0 0 0))
+  )
   (wire (pts (xy 140.97 34.29) (xy 140.97 36.83))
     (stroke (width 0) (type default) (color 0 0 0 0))
@@
     (stroke (width 0) (type default) (color 0 0 0 0))
   )
+  (wire (pts (xy 160.274 86.614) (xy 160.274 92.964))
+    (stroke (width 0) (type default) (color 0 0 0 0))
+  )
   (wire (pts (xy 130.81 26.67) (xy 130.81 21.59))
     (stroke (width 0) (type default) (color 0 0 0 0))
@@
     (stroke (width 0) (type default) (color 0 0 0 0))
   )
+  (wire (pts (xy 156.464 84.074) (xy 150.114 84.074))
+    (stroke (width 0) (type default) (color 0 0 0 0))
+  )
   (wire (pts (xy 246.38 102.87) (xy 246.38 95.25))
     (stroke (width 0) (type default) (color 0 0 0 0))
@@
     (stroke (width 0) (type default) (color 0 0 0 0))
   )
+  (wire (pts (xy 156.464 70.104) (xy 150.114 70.104))
+    (stroke (width 0) (type default) (color 0 0 0 0))
+  )
   (wire (pts (xy 113.03 102.87) (xy 113.03 96.52))
     (stroke (width 0) (type default) (color 0 0 0 0))
@@
     (effects (font (size 1.27 1.27)) (justify left bottom))
   )
+  (text "Pluviomètre" (at 125.73 108.204 0)
+    (effects (font (size 1.27 1.27)) (justify left bottom))
+  )
   (text "GPS" (at 15.24 153.67 0)
     (effects (font (size 1.27 1.27)) (justify left bottom))
@@
     )
   )
+  (global_label "+3V3" (shape input) (at 150.114 70.104 180) (fields_autoplaced)
+    (effects (font (size 1.27 1.27)) (justify right))
+    (property "Intersheet References" "${INTERSHEET_REFS}" (id 0) (at -40.386 -58.166 0)
+      (effects (font (size 1.27 1.27)) hide)
+    )
+  )
+  (global_label "Rain_gauge" (shape output) (at 150.114 84.074 180) (fields_autoplaced)
+    (effects (font (size 1.27 1.27)) (justify right))
+    (property "Intersheet References" "${INTERSHEET_REFS}" (id 0) (at 136.9646 83.9946 0)
+      (effects (font (size 1.27 1.27)) (justify right) hide)
+    )
+  )
   (global_label "SDA" (shape bidirectional) (at 187.96 120.65 0) (fields_autoplaced)
     (effects (font (size 1.27 1.27)) (justify left))
@@
     (pin "1")
   )
+  (symbol (lib_id "Device:R") (at 156.464 76.454 0) (unit 1)
+    (in_bom yes) (on_board yes)
+    (property "Reference" "R43" (id 0) (at 158.242 75.2856 0)
+      (effects (font (size 1.27 1.27)) (justify left))
+    )
+    (property "Value" "100k" (id 1) (at 158.242 77.597 0)
+      (effects (font (size 1.27 1.27)) (justify left))
+    )
+    (property "Footprint" "Resistor_SMD:R_0603_1608Metric" (id 2) (at 154.686 76.454 90)
+      (effects (font (size 1.27 1.27)) hide)
+    )
+    (property "Datasheet" "~" (id 3) (at 156.464 76.454 0)
+      (effects (font (size 1.27 1.27)) hide)
+    )
+    (pin "1")
+    (pin "2")
+  )
+  (symbol (lib_id "power:GND") (at 160.274 92.964 0) (unit 1)
+    (in_bom yes) (on_board yes)
+    (property "Reference" "#PWR0232" (id 0) (at 160.274 99.314 0)
+      (effects (font (size 1.27 1.27)) hide)
+    )
+    (property "Value" "GND" (id 1) (at 160.401 97.3582 0))
+    (property "Footprint" "" (id 2) (at 160.274 92.964 0)
+      (effects (font (size 1.27 1.27)) hide)
+    )
+    (property "Datasheet" "" (id 3) (at 160.274 92.964 0)
+      (effects (font (size 1.27 1.27)) hide)
+    )
+    (pin "1")
+  )
   (symbol (lib_id "Device:R") (at 226.06 110.49 270) (unit 1)
     (in_bom yes) (on_board yes)
@@
     (pin "2")
   )
+  (symbol (lib_id "Connector_Generic:Conn_01x02") (at 172.974 84.074 0) (unit 1)
+    (in_bom yes) (on_board yes)
+    (property "Reference" "J21" (id 0) (at 175.006 84.2772 0)
+      (effects (font (size 1.27 1.27)) (justify left))
+    )
+    (property "Value" "Conn_01x02" (id 1) (at 175.006 86.5886 0)
+      (effects (font (size 1.27 1.27)) (justify left))
+    )
+    (property "Footprint" "Connector_JST:JST_PH_B2B-PH-K_1x02_P2.00mm_Vertical" (id 2) (at 172.974 84.074 0)
+      (effects (font (size 1.27 1.27)) hide)
+    )
+    (property "Datasheet" "~" (id 3) (at 172.974 84.074 0)
+      (effects (font (size 1.27 1.27)) hide)
+    )
+    (pin "1")
+    (pin "2")
+  )
   (symbol (lib_id "power:GND") (at 140.97 36.83 0) (unit 1)
     (in_bom yes) (on_board yes)
@@
       (reference "#PWR0231") (unit 1) (value "GND") (footprint "")
     )
+    (path "/50b2a9a4-4d9d-4c61-baa0-7977acbd17d1"
+      (reference "#PWR0232") (unit 1) (value "GND") (footprint "")
+    )
     (path "/00000000-0000-0000-0000-0000609e7af1/bb7ae7f6-63de-450d-ae2b-f3b6c8a246d5"
       (reference "#PWR0234") (unit 1) (value "GND") (footprint "")
@@
       (reference "J20") (unit 1) (value "USB_C_Receptacle_USB2.0 USB4105-GF-A ") (footprint "Empreintes:TYPE-C-31-M-12")
     )
+    (path "/534352b5-344f-40fd-9b86-d6a504145924"
+      (reference "J21") (unit 1) (value "Conn_01x02") (footprint "Connector_JST:JST_PH_B2B-PH-K_1x02_P2.00mm_Vertical")
+    )
     (path "/00000000-0000-0000-0000-00006011445d/79fe9980-abb4-43ab-a32a-a54b421cb267"
       (reference "JP1") (unit 1) (value "SolderJumper_3_Open") (footprint "Jumper:SolderJumper-3_P1.3mm_Open_RoundedPad1.0x1.5mm_NumberLabels")
@@
       (reference "R42") (unit 1) (value "499/5%") (footprint "Resistor_SMD:R_0603_1608Metric")
     )
+    (path "/4dd3a74b-b6c6-4867-9d42-187bc415bbf2"
+      (reference "R43") (unit 1) (value "100k") (footprint "Resistor_SMD:R_0603_1608Metric")
+    )
     (path "/a9a1feef-c39d-4052-8bf2-e3ffc2216412/40bc5463-a30d-4b86-89ed-b91c5a12ef42"

Commit message: Update
Other:
- note added: "External RESET push button"
- note added: "Heltec Wireless shell V3 POWER SUPPLY"
Changed lines of the file:
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@@
   (title_block
     (title "Open_beehive_scale_board")
-    (date "2022-05-16")
-    (rev "V0.1")
+    (date "2023-01-13")
+    (rev "V0.4")
     (company "Ratamuse")
   )
@@
     (effects (font (size 1.27 1.27)) (justify left bottom))
   )
-  (text "Battery supervision\n" (at 124.46 151.13 0)
+  (text "Battery supervision\n" (at 124.714 155.448 0)
+    (effects (font (size 1.27 1.27)) (justify left bottom))
+  )
+  (text "Heltec Wireless shell V3 POWER SUPPLY" (at 124.968 53.086 0)
     (effects (font (size 1.27 1.27)) (justify left bottom))
   )
@@
     (effects (font (size 1.27 1.27)) (justify left bottom))
   )
+  (text "External RESET push button" (at 126.492 195.326 0)
+    (effects (font (size 1.27 1.27)) (justify left bottom))
+  )
   (text "Pressure sensor" (at 200.66 116.84 0)
     (effects (font (size 1.27 1.27)) (justify left bottom))
@@
       (reference "#PWR0126") (unit 1) (value "GND") (footprint "")
     )
-    (path "/00000000-0000-0000-0000-00006011445d/9d6c492f-a56c-4a47-99a2-4fcd0c43c5ec"
+    (path "/a9a1feef-c39d-4052-8bf2-e3ffc2216412/63fea5a4-61b5-44d3-9907-b5f7d4c10d2f"
       (reference "#PWR0127") (unit 1) (value "GND") (footprint "")
     )
@@
       (reference "#PWR0232") (unit 1) (value "GND") (footprint "")
     )
+    (path "/00000000-0000-0000-0000-00006011445d/c02a9f41-7766-4886-9874-3c122de45fa2"
+      (reference "#PWR0233") (unit 1) (value "GND") (footprint "")
+    )
     (path "/00000000-0000-0000-0000-0000609e7af1/bb7ae7f6-63de-450d-ae2b-f3b6c8a246d5"
       (reference "#PWR0234") (unit 1) (value "GND") (footprint "")
@@
       (reference "C64") (unit 1) (value "0.1µF") (footprint "Capacitor_SMD:C_0603_1608Metric")
     )
+    (path "/a9a1feef-c39d-4052-8bf2-e3ffc2216412/18e9bf14-e16c-4d39-834c-de3b592af806"
+      (reference "C65") (unit 1) (value "0.1µF") (footprint "Capacitor_SMD:C_0805_2012Metric")
+    )
     (path "/00000000-0000-0000-0000-0000609e7af1/20fa6fea-0ecc-4b67-b8cc-6a4de1a0d2a6"
       (reference "D1") (unit 1) (value "LED") (footprint "LED_SMD:LED_0603_1608Metric_Castellated")
@@
       (reference "J3") (unit 1) (value "Conn_01x03") (footprint "Connector_JST:JST_PH_B3B-PH-K_1x03_P2.00mm_Vertical")
     )
-    (path "/00000000-0000-0000-0000-00006011445d/5d24980b-7611-49f9-b4eb-245894554c4b"
-      (reference "J4") (unit 1) (value "Conn_01x03") (footprint "Connector_JST:JST_PH_B3B-PH-K_1x03_P2.00mm_Vertical")
+    (path "/00000000-0000-0000-0000-00006011445d/04077ed3-6466-4148-9df4-ea025f279428"
+      (reference "J4") (unit 1) (value "Conn_01x02") (footprint "Connector_JST:JST_PH_B2B-PH-K_1x02_P2.00mm_Vertical")
     )
     (path "/00000000-0000-0000-0000-00006011445d/e8787f64-d77a-42cc-a9f5-8346c8d80077"
@@
       (reference "J21") (unit 1) (value "Conn_01x02") (footprint "Connector_JST:JST_PH_B2B-PH-K_1x02_P2.00mm_Vertical")
     )
-    (path "/00000000-0000-0000-0000-00006011445d/79fe9980-abb4-43ab-a32a-a54b421cb267"
-      (reference "JP1") (unit 1) (value "SolderJumper_3_Open") (footprint "Jumper:SolderJumper-3_P1.3mm_Open_RoundedPad1.0x1.5mm_NumberLabels")
-    )
     (path "/00000000-0000-0000-0000-0000609e7af1/d3ebbd18-8772-4e3c-a3ab-aa9dd5493a54"
       (reference "L1") (unit 1) (value "82µH/3A") (footprint "Empreintes:INDPM138126X700N")
@@
       (reference "R53") (unit 1) (value "100") (footprint "Resistor_SMD:R_0603_1608Metric")
     )
+    (path "/a9a1feef-c39d-4052-8bf2-e3ffc2216412/1791033d-8643-4d87-bec8-492e0cfae666"
+      (reference "R54") (unit 1) (value "10K") (footprint "Resistor_SMD:R_0603_1608Metric")
+    )
     (path "/00000000-0000-0000-0000-000062773850"
       (reference "S1") (unit 1) (value "RB231X2") (footprint "Empreintes:RB231X2")
@@
       (reference "SW1") (unit 1) (value "SW_Push") (footprint "Empreintes:PTS636SL43SMTRLFS")
     )
+    (path "/a9a1feef-c39d-4052-8bf2-e3ffc2216412/47a88e7c-4b09-4fe1-9cff-053d8d879663"
+      (reference "SW2") (unit 1) (value "SW_Push") (footprint "Empreintes:PTS636SL43SMTRLFS")
+    )
     (path "/a9a1feef-c39d-4052-8bf2-e3ffc2216412/e34719be-30e8-4756-8475-8be71c8100da"
       (reference "U1") (unit 1) (value "CP2102N-A02-GQFN24") (footprint "Package_DFN_QFN:QFN-24-1EP_4x4mm_P0.5mm_EP2.6x2.6mm")
@@
       (reference "U6") (unit 1) (value "Heltec_Wireless_shell_V3") (footprint "Empreintes:Heltec Wireless shell V3")
     )
-    (path "/00000000-0000-0000-0000-0000609e7af1/f526b5d4-d24d-4a26-ba08-bbacc53ec371"
+    (path "/00000000-0000-0000-0000-00006011445d/cb63f569-c9cd-49a5-aaa0-53a6c6aafd1d"
       (reference "U7") (unit 1) (value "1043") (footprint "Empreintes:1043")
     )

Commit message: Update
Parts:
- C51, C60: footprint Capacitor_SMD:C_0603_1608Metric -> Capacitor_SMD:C_0805_2012Metric
- C52, C61: footprint Capacitor_SMD:C_0805_2012Metric -> Capacitor_SMD:C_0603_1608Metric
Changed lines of the file:
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@@
       (effects (font (size 1.27 1.27)) (justify left))
     )
-    (property "Footprint" "Capacitor_SMD:C_0603_1608Metric" (id 2) (at 131.7752 34.29 0)
+    (property "Footprint" "Capacitor_SMD:C_0805_2012Metric" (id 2) (at 131.7752 34.29 0)
       (effects (font (size 1.27 1.27)) hide)
     )
@@
       (effects (font (size 1.27 1.27)) (justify left))
     )
-    (property "Footprint" "Capacitor_SMD:C_0603_1608Metric" (id 2) (at 41.6052 36.83 0)
+    (property "Footprint" "Capacitor_SMD:C_0805_2012Metric" (id 2) (at 41.6052 36.83 0)
       (effects (font (size 1.27 1.27)) hide)
     )
@@
       (effects (font (size 1.27 1.27)) (justify left))
     )
-    (property "Footprint" "Capacitor_SMD:C_0805_2012Metric" (id 2) (at 141.9352 34.29 0)
+    (property "Footprint" "Capacitor_SMD:C_0603_1608Metric" (id 2) (at 141.9352 34.29 0)
       (effects (font (size 1.27 1.27)) hide)
     )
@@
       (effects (font (size 1.27 1.27)) (justify left))
     )
-    (property "Footprint" "Capacitor_SMD:C_0805_2012Metric" (id 2) (at 51.7652 36.83 0)
+    (property "Footprint" "Capacitor_SMD:C_0603_1608Metric" (id 2) (at 51.7652 36.83 0)
       (effects (font (size 1.27 1.27)) hide)
     )
@@
     )
     (path "/4bd821f2-0707-4078-b490-ee80c8fe83b7"
-      (reference "C51") (unit 1) (value "10µF") (footprint "Capacitor_SMD:C_0603_1608Metric")
+      (reference "C51") (unit 1) (value "10µF") (footprint "Capacitor_SMD:C_0805_2012Metric")
     )
     (path "/fd8286f5-83f2-4c75-b09d-fdd0c502a928"
-      (reference "C52") (unit 1) (value "0.1µF") (footprint "Capacitor_SMD:C_0805_2012Metric")
+      (reference "C52") (unit 1) (value "0.1µF") (footprint "Capacitor_SMD:C_0603_1608Metric")
     )
     (path "/d2746501-2960-4618-ba16-fa886c4044e2"
@@
     )
     (path "/3be1f3e2-daac-4308-97d4-8357e9694a12"
-      (reference "C60") (unit 1) (value "10µF") (footprint "Capacitor_SMD:C_0603_1608Metric")
+      (reference "C60") (unit 1) (value "10µF") (footprint "Capacitor_SMD:C_0805_2012Metric")
     )
     (path "/f9f6873b-1e72-4d7c-9757-607196772c1e"
-      (reference "C61") (unit 1) (value "0.1µF") (footprint "Capacitor_SMD:C_0805_2012Metric")
+      (reference "C61") (unit 1) (value "0.1µF") (footprint "Capacitor_SMD:C_0603_1608Metric")
     )
     (path "/708d242d-c3e5-4d5d-8b27-4d2d23416d33"
@@
     )
     (path "/a9a1feef-c39d-4052-8bf2-e3ffc2216412/18e9bf14-e16c-4d39-834c-de3b592af806"
-      (reference "C65") (unit 1) (value "0.1µF") (footprint "Capacitor_SMD:C_0805_2012Metric")
+      (reference "C65") (unit 1) (value "0.1µF") (footprint "Capacitor_SMD:C_0603_1608Metric")
     )
     (path "/00000000-0000-0000-0000-0000609e7af1/20fa6fea-0ecc-4b67-b8cc-6a4de1a0d2a6"
@@
     )
     (path "/00000000-0000-0000-0000-0000609e7af1/26b8040d-b4b6-44ec-9538-7e7484d33d9d"
-      (reference "R1") (unit 1) (value "2K") (footprint "Resistor_SMD:R_0603_1608Metric")
+      (reference "R1") (unit 1) (value "10K") (footprint "Resistor_SMD:R_0603_1608Metric")
     )
     (path "/00000000-0000-0000-0000-0000609e7af1/0e7d6f7e-cab7-471f-bbc4-637272e771c1"
