File: ruchea.kicad_sch (KiCad schematic)
At the start: 25 parts, among them J11 Conn_01x04, J12 Conn_01x04, J14 Conn_01x03, J17 Conn_01x04, J18 Conn_01x04, J3 Conn_01x03, J4 Conn_01x03, J5 Conn_01x04, J8 Conn_01x03, J9 Conn_01x03, U4 TCA9548APWR

Commit message: Update
Parts:
- removed J4: Conn_01x03, Connector_JST:JST_PH_B3B-PH-K_1x03_P2.00mm_Vertical, symbol Connector_Generic:Conn_01x03
- removed JP1: SolderJumper_3_Open, Jumper:SolderJumper-3_P1.3mm_Open_RoundedPad1.0x1.5mm_NumberLabels, symbol ruche-rescue:SolderJumper_3_Open-Jumper
- added J4: Conn_01x02, Connector_JST:JST_PH_B2B-PH-K_1x02_P2.00mm_Vertical, symbol Connector_Generic:Conn_01x02
- added U7: 1043, Empreintes:1043, symbol 1043:1043
Connections:
- net GND: now also J4.2 (Pin_2)
- new net VBAT: J4.1 (Pin_1), U7.1 (+)
- new net VBAT-: U7.2 (-)
Other:
- note added: "I2C multiplexor"
- note added: "Scale 1"
- note added: "Scale 2"
- note added: "Scale 3"
- note added: "Scale 4"
- moved on the sheet: J17
