File: rucheb.kicad_sch (KiCad schematic)
At the start: 29 parts, among them IC1 CN3791, IC9 FS312F-G, J1 Conn_01x02, Q1 AO3401A, Q8 FS8205, U7 1043

Commit message: Update
Parts:
- removed U7: 1043, Empreintes:1043, symbol 1043:1043
Changed lines of the file:
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@@
   (title_block
     (title "Open_beehive_scale_board")
-    (date "2022-05-16")
-    (rev "V0.1")
+    (date "2023-01-13")
+    (rev "V0.4")
     (company "Ratamuse")
   )
@@
     (stroke (width 0) (type default) (color 0 0 0 0))
   )
-  (wire (pts (xy 232.41 153.67) (xy 243.84 153.67))
-    (stroke (width 0) (type default) (color 0 0 0 0))
-  )
   (wire (pts (xy 187.96 81.28) (xy 194.31 81.28))
     (stroke (width 0) (type default) (color 0 0 0 0))
@@
   )
   (wire (pts (xy 91.44 120.65) (xy 91.44 116.84))
-    (stroke (width 0) (type default) (color 0 0 0 0))
-  )
-  (wire (pts (xy 232.41 151.13) (xy 243.84 151.13))
     (stroke (width 0) (type default) (color 0 0 0 0))
   )
@@
     )
   )
-  (global_label "VBAT" (shape input) (at 232.41 151.13 180) (fields_autoplaced)
-    (effects (font (size 1.27 1.27)) (justify right))
-    (property "Intersheet References" "${INTERSHEET_REFS}" (id 0) (at 225.671 151.0506 0)
-      (effects (font (size 1.27 1.27)) (justify right) hide)
-    )
-  )
   (global_label "VBAT" (shape output) (at 273.05 40.64 0) (fields_autoplaced)
     (effects (font (size 1.27 1.27)) (justify left))
@@
     (property "Intersheet References" "${INTERSHEET_REFS}" (id 0) (at 22.86 -58.42 0)
       (effects (font (size 1.27 1.27)) hide)
-    )
-  )
-  (global_label "VBAT-" (shape input) (at 232.41 153.67 180) (fields_autoplaced)
-    (effects (font (size 1.27 1.27)) (justify right))
-    (property "Intersheet References" "${INTERSHEET_REFS}" (id 0) (at 224.0987 153.5906 0)
-      (effects (font (size 1.27 1.27)) (justify right) hide)
     )
   )
@@
     (pin "1")
   )
-  (symbol (lib_id "1043:1043") (at 243.84 151.13 0) (unit 1)
-    (in_bom yes) (on_board yes) (fields_autoplaced)
-    (property "Reference" "U7" (id 0) (at 256.54 144.941 0))
-    (property "Value" "1043" (id 1) (at 256.54 147.4779 0))
-    (property "Footprint" "Empreintes:1043" (id 2) (at 265.43 148.59 0)
-      (effects (font (size 1.27 1.27)) (justify left) hide)
-    )
-    (property "Datasheet" "http://www.keyelco.com/product-pdf.cfm?p=919" (id 3) (at 265.43 151.13 0)
-      (effects (font (size 1.27 1.27)) (justify left) hide)
-    )
-    (property "Description" "KEYSTONE - 1043 - BATTERY HOLDER, 18650, TH" (id 4) (at 265.43 153.67 0)
-      (effects (font (size 1.27 1.27)) (justify left) hide)
-    )
-    (property "Height" "14.86" (id 5) (at 265.43 156.21 0)
-      (effects (font (size 1.27 1.27)) (justify left) hide)
-    )
-    (property "Mouser Part Number" "534-1043" (id 6) (at 265.43 158.75 0)
-      (effects (font (size 1.27 1.27)) (justify left) hide)
-    )
-    (property "Mouser Price/Stock" "https://www.mouser.co.uk/ProductDetail/Keystone-Electronics/1043?qs=%2F7TOpeL5Mz6j%2FnxeOA1rsg%3D%3D" (id 7) (at 265.43 161.29 0)
-      (effects (font (size 1.27 1.27)) (justify left) hide)
-    )
-    (property "Manufacturer_Name" "Keystone Electronics" (id 8) (at 265.43 163.83 0)
-      (effects (font (size 1.27 1.27)) (justify left) hide)
-    )
-    (property "Manufacturer_Part_Number" "1043" (id 9) (at 265.43 166.37 0)
-      (effects (font (size 1.27 1.27)) (justify left) hide)
-    )
-    (pin "1")
-    (pin "2")
-    (pin "MH1")
-    (pin "MH2")
-    (pin "MH3")
-  )
 )

Commit message: Update
Parts:
- R1: value 2K -> 10K
Changed lines of the file:
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@@
       (effects (font (size 1.27 1.27)) (justify left))
     )
-    (property "Value" "2K" (id 1) (at 34.798 76.073 0)
+    (property "Value" "10K" (id 1) (at 34.798 76.073 0)
       (effects (font (size 1.27 1.27)) (justify left))
     )
