File: ruched.kicad_sch (KiCad schematic)
At the start: 23 parts, among them J20 USB_C_Receptacle_USB2.0 USB41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, Q6 UMH3N, Q7 DMG2301L, SW1 SW_Push, U1 CP2102N-A02-GQFN24

Commit message: Update
Parts:
- removed U?: Heltec_Wifi_LoRa_V3, symbol Espressif:Heltec_Wifi_LoRa_V3
- added R42: 499/5%, Resistor_SMD:R_0603_1608Metric, symbol Device:R
- added U6: Heltec_Wireless_shell_V3, Empreintes:Heltec Wireless shell V3, symbol Espressif:Heltec_Wireless_shell_V3
Connections:
- net CLK-SCK-D9: now also U6.13 (GPIO41)
- net CLK1: now also U6.28 (GPIO18)
- net CLK2: now also U6.29 (GPIO20)
- net CLK3: now also U6.31 (GPIO17)
- net CLK4: now also U6.5 (GPIO33)
- net CMD-MOSI-D8: now also U6.12 (GPIO40)
- net DAT1: now also U6.10 (GPIO38)
- net DAT2: now also U6.25 (GPIO7)
- net DAT3: now also U6.32 (GPIO19)
- net DAT4: now also U6.6 (GPIO34)
- net DS18b20: now also U6.24 (GPIO6)
- net EN: now also U6.23 (EN)
- net GND: now also U6.41 (Gnd), U6.42 (Gnd), U6.43 (Gnd), U6.44 (Gnd)
- net INT1: now also U6.21 (GPIO2)
- net IO0: now also U6.34 (GPIO0)
- net RX_GPS: now also U6.17 (GPIO45)
- net SCL: now also U6.36 (GPIO4)
- net SD3-CS-D7: now also U6.14 (GPIO42)
- net SDA: now also U6.35 (GPIO5)
- net SDO-MISO-D10: now also U6.11 (GPIO39)
- net Start_GPS: now also U6.8 (GPIO36)
- net Start_modules: now also U6.9 (GPIO37)
- net TX_GPS: now also U6.18 (GPIO46)
- net Tilt_led_alarm: now also U6.7 (GPIO35)
- net UORXD: now also U6.15 (RXD)
- net UOTXD: now also R42.2
- new net: R42.1, U6.16 (TXD)
- new net: U6.3 (3V3), U6.4 (3V3)

Commit message: Update
Connections:
- net +3V3: now also U6.3 (3V3), U6.4 (3V3)
- net CLK1: now also U6.6 (GPIO34); no longer U6.28 (GPIO18)
- net CLK2: now also U6.7 (GPIO35); no longer U6.29 (GPIO20)
- net CLK3: now also U6.25 (GPIO7); no longer U6.31 (GPIO17)
- net CLK4: now also U6.20 (GPIO1); no longer U6.5 (GPIO33)
- net DAT1: now also U6.5 (GPIO33); no longer U6.10 (GPIO38)
- net DAT2: now also U6.9 (GPIO37); no longer U6.25 (GPIO7)
- net DAT3: now also U6.24 (GPIO6); no longer U6.32 (GPIO19)
- net DAT4: now also U6.21 (GPIO2); no longer U6.6 (GPIO34)
- net DS18b20: now also U6.33 (GPIO21); no longer U6.24 (GPIO6)
- net INT1: now also U6.27 (GPIO16); no longer U6.21 (GPIO2)
- net Start_GPS: now also U6.26 (GPIO15); no longer U6.8 (GPIO36)
- net Start_modules: now also U6.28 (GPIO18); no longer U6.9 (GPIO37)
- net Tilt_led_alarm: now also U6.8 (GPIO36/Vext_Ctrl); no longer U6.7 (GPIO35)
- new net Rain_gauge: U6.31 (GPIO17)

Commit message: Update
Connections:
- net CLK1: now also U6.22 (GPIO3); no longer U6.6 (GPIO34)
- net DAT1: now also U6.10 (GPIO38); no longer U6.5 (GPIO33)
Other:
- moved on the sheet: R42
Changed lines of the file:
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@@
     (stroke (width 0) (type default) (color 0 0 0 0))
   )
-  (wire (pts (xy 143.256 39.878) (xy 167.64 39.878))
+  (wire (pts (xy 149.606 39.878) (xy 167.64 39.878))
     (stroke (width 0) (type default) (color 0 0 0 0))
   )
@@
     (stroke (width 0) (type default) (color 0 0 0 0))
   )
-  (wire (pts (xy 130.556 39.878) (xy 135.636 39.878))
+  (wire (pts (xy 138.43 39.878) (xy 141.986 39.878))
     (stroke (width 0) (type default) (color 0 0 0 0))
   )
@@
     (stroke (width 0) (type default) (color 0 0 0 0))
   )
-  (wire (pts (xy 159.258 67.818) (xy 167.64 67.818))
-    (stroke (width 0) (type default) (color 0 0 0 0))
-  )
   (wire (pts (xy 63.5 25.4) (xy 68.58 25.4))
     (stroke (width 0) (type default) (color 0 0 0 0))
@@
     (stroke (width 0) (type default) (color 0 0 0 0))
   )
-  (wire (pts (xy 159.258 65.278) (xy 167.64 65.278))
+  (wire (pts (xy 159.258 24.638) (xy 167.64 24.638))
     (stroke (width 0) (type default) (color 0 0 0 0))
   )
@@
     (stroke (width 0) (type default) (color 0 0 0 0))
   )
+  (wire (pts (xy 159.258 55.118) (xy 167.386 55.118))
+    (stroke (width 0) (type default) (color 0 0 0 0))
+  )
   (wire (pts (xy 166.624 72.39) (xy 167.64 72.39))
     (stroke (width 0) (type default) (color 0 0 0 0))
@@
     )
   )
-  (global_label "Rain_gauge" (shape output) (at 246.634 44.958 0) (fields_autoplaced)
+  (global_label "Rain_gauge" (shape input) (at 246.634 44.958 0) (fields_autoplaced)
     (effects (font (size 1.27 1.27)) (justify left))
     (property "Intersheet References" "${INTERSHEET_REFS}" (id 0) (at 259.7834 44.8786 0)
@@
     )
   )
-  (global_label "CLK1" (shape bidirectional) (at 159.258 65.278 180) (fields_autoplaced)
-    (effects (font (size 1.27 1.27)) (justify right))
-    (property "Intersheet References" "${INTERSHEET_REFS}" (id 0) (at 152.1562 65.1986 0)
+  (global_label "CLK1" (shape bidirectional) (at 159.258 24.638 180) (fields_autoplaced)
+    (effects (font (size 1.27 1.27)) (justify right))
+    (property "Intersheet References" "${INTERSHEET_REFS}" (id 0) (at 152.1562 24.5586 0)
       (effects (font (size 1.27 1.27)) (justify right) hide)
     )
@@
     )
   )
-  (global_label "UOTXD" (shape output) (at 130.556 39.878 180) (fields_autoplaced)
-    (effects (font (size 1.27 1.27)) (justify right))
-    (property "Intersheet References" "${INTERSHEET_REFS}" (id 0) (at 122.1237 39.7986 0)
+  (global_label "UOTXD" (shape output) (at 138.43 39.878 180) (fields_autoplaced)
+    (effects (font (size 1.27 1.27)) (justify right))
+    (property "Intersheet References" "${INTERSHEET_REFS}" (id 0) (at 129.9977 39.7986 0)
       (effects (font (size 1.27 1.27)) (justify right) hide)
     )
@@
     )
   )
-  (global_label "DAT1" (shape bidirectional) (at 159.258 67.818 180) (fields_autoplaced)
-    (effects (font (size 1.27 1.27)) (justify right))
-    (property "Intersheet References" "${INTERSHEET_REFS}" (id 0) (at 152.3981 67.7386 0)
+  (global_label "DAT1" (shape bidirectional) (at 159.258 55.118 180) (fields_autoplaced)
+    (effects (font (size 1.27 1.27)) (justify right))
+    (property "Intersheet References" "${INTERSHEET_REFS}" (id 0) (at 152.3981 55.0386 0)
       (effects (font (size 1.27 1.27)) (justify right) hide)
     )
@@
     (pin "1")
   )
-  (symbol (lib_id "Device:R") (at 139.446 39.878 270) (unit 1)
-    (in_bom yes) (on_board yes)
-    (property "Reference" "R42" (id 0) (at 139.446 34.6202 90))
-    (property "Value" "499/5%" (id 1) (at 139.446 36.9316 90))
-    (property "Footprint" "Resistor_SMD:R_0603_1608Metric" (id 2) (at 139.446 38.1 90)
-      (effects (font (size 1.27 1.27)) hide)
-    )
-    (property "Datasheet" "~" (id 3) (at 139.446 39.878 0)
-      (effects (font (size 1.27 1.27)) hide)
-    )
+  (symbol (lib_id "Device:R") (at 145.796 39.878 270) (unit 1)
+    (in_bom yes) (on_board yes)
+    (property "Reference" "R42" (id 0) (at 145.796 34.6202 90))
+    (property "Value" "499/5%" (id 1) (at 145.796 36.9316 90))
+    (property "Footprint" "Resistor_SMD:R_0603_1608Metric" (id 2) (at 145.796 38.1 90)
+      (effects (font (size 1.27 1.27)) hide)
+    )
+    (property "Datasheet" "~" (id 3) (at 145.796 39.878 0)
+      (effects (font (size 1.27 1.27)) hide)
+    )

Commit message: Update
Parts:
- added C65: 0.1µF, Capacitor_SMD:C_0805_2012Metric, symbol Device:C
- added R54: 10K, Resistor_SMD:R_0603_1608Metric, symbol Device:R
- added SW2: SW_Push, Empreintes:PTS636SL43SMTRLFS, symbol Switch:SW_Push
Connections:
- net +3V3: now also R54.1
- net DTR: now also C65.2
- net EN: now also C65.1
- net GND: now also SW2.2
- net IO0: now also R54.2, SW2.1
Other:
- company: (none) -> Ratamuse
- title: (none) -> Open_beehive_scale_board
- moved on the sheet: C57, C58, C59, D14, Q6, Q7, R48, R49, SW1

Commit message: Update
Parts:
- C65: footprint Capacitor_SMD:C_0805_2012Metric -> Capacitor_SMD:C_0603_1608Metric
Changed lines of the file:
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@@
       (effects (font (size 1.27 1.27)) (justify left))
     )
-    (property "Footprint" "Capacitor_SMD:C_0805_2012Metric" (id 2) (at 230.8352 130.81 0)
+    (property "Footprint" "Capacitor_SMD:C_0603_1608Metric" (id 2) (at 230.8352 130.81 0)
       (effects (font (size 1.27 1.27)) hide)
     )

Commit message: Update
Connections:
- net CLK1: now also U6.26 (GPIO15); no longer U6.22 (GPIO3)
- net CLK2: now also U6.38 (GPIO47); no longer U6.7 (GPIO35)
- net CLK3: now also U6.24 (GPIO6); no longer U6.25 (GPIO7)
- net CLK4: now also U6.22 (GPIO3); no longer U6.20 (GPIO1)
- net DAT1: now also U6.35 (GPIO5); no longer U6.10 (GPIO38)
- net DAT2: now also U6.36 (GPIO4); no longer U6.9 (GPIO37)
- net DAT3: now also U6.25 (GPIO7); no longer U6.24 (GPIO6)
- net DS18b20: now also U6.7 (GPIO35); no longer U6.33 (GPIO21)
- net SCL: now also U6.9 (GPIO37); no longer U6.36 (GPIO4)
- net SDA: now also U6.10 (GPIO38); no longer U6.35 (GPIO5)
- net Start_GPS: now also U6.20 (GPIO1); no longer U6.26 (GPIO15)
Changed lines of the file:
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@@
+    (stroke (width 0) (type default) (color 0 0 0 0))
+  )
+  (wire (pts (xy 241.554 62.738) (xy 247.396 62.738))
     (stroke (width 0) (type default) (color 0 0 0 0))
   )
@@
     (stroke (width 0) (type default) (color 0 0 0 0))
   )
+  (wire (pts (xy 159.512 62.738) (xy 167.64 62.738))
+    (stroke (width 0) (type default) (color 0 0 0 0))
+  )
   (wire (pts (xy 63.5 25.4) (xy 68.58 25.4))
     (stroke (width 0) (type default) (color 0 0 0 0))
@@
     (stroke (width 0) (type default) (color 0 0 0 0))
   )
-  (wire (pts (xy 159.258 62.738) (xy 167.64 62.738))
-    (stroke (width 0) (type default) (color 0 0 0 0))
-  )
   (wire (pts (xy 48.26 38.1) (xy 48.26 25.4))
     (stroke (width 0) (type default) (color 0 0 0 0))
@@
     (stroke (width 0) (type default) (color 0 0 0 0))
   )
-  (wire (pts (xy 241.554 50.038) (xy 247.396 50.038))
-    (stroke (width 0) (type default) (color 0 0 0 0))
-  )
   (wire (pts (xy 86.36 106.68) (xy 86.36 102.87))
     (stroke (width 0) (type default) (color 0 0 0 0))
@@
     )
   )
-  (global_label "CLK3" (shape bidirectional) (at 245.872 29.718 0) (fields_autoplaced)
-    (effects (font (size 1.27 1.27)) (justify left))
-    (property "Intersheet References" "${INTERSHEET_REFS}" (id 0) (at 252.9738 29.6386 0)
+  (global_label "DAT3" (shape bidirectional) (at 245.872 29.718 0) (fields_autoplaced)
+    (effects (font (size 1.27 1.27)) (justify left))
+    (property "Intersheet References" "${INTERSHEET_REFS}" (id 0) (at 252.7319 29.6386 0)
       (effects (font (size 1.27 1.27)) (justify left) hide)
     )
@@
     )
   )
-  (global_label "SDA" (shape bidirectional) (at 247.396 55.118 0) (fields_autoplaced)
-    (effects (font (size 1.27 1.27)) (justify left))
-    (property "Intersheet References" "${INTERSHEET_REFS}" (id 0) (at 253.2883 55.0386 0)
+  (global_label "DAT1" (shape bidirectional) (at 247.396 55.118 0) (fields_autoplaced)
+    (effects (font (size 1.27 1.27)) (justify left))
+    (property "Intersheet References" "${INTERSHEET_REFS}" (id 0) (at 254.2559 55.0386 0)
       (effects (font (size 1.27 1.27)) (justify left) hide)
     )
@@
     )
   )
-  (global_label "CLK2" (shape bidirectional) (at 159.258 62.738 180) (fields_autoplaced)
-    (effects (font (size 1.27 1.27)) (justify right))
-    (property "Intersheet References" "${INTERSHEET_REFS}" (id 0) (at 152.1562 62.6586 0)
-      (effects (font (size 1.27 1.27)) (justify right) hide)
+  (global_label "CLK2" (shape bidirectional) (at 247.396 62.738 0) (fields_autoplaced)
+    (effects (font (size 1.27 1.27)) (justify left))
+    (property "Intersheet References" "${INTERSHEET_REFS}" (id 0) (at 254.4978 62.6586 0)
+      (effects (font (size 1.27 1.27)) (justify left) hide)
     )
   )
@@
     )
   )
-  (global_label "CLK1" (shape bidirectional) (at 159.258 24.638 180) (fields_autoplaced)
+  (global_label "CLK4" (shape bidirectional) (at 159.258 24.638 180) (fields_autoplaced)
     (effects (font (size 1.27 1.27)) (justify right))
     (property "Intersheet References" "${INTERSHEET_REFS}" (id 0) (at 152.1562 24.5586 0)
@@
     )
   )
-  (global_label "Start_GPS" (shape output) (at 246.634 32.258 0) (fields_autoplaced)
-    (effects (font (size 1.27 1.27)) (justify left))
-    (property "Intersheet References" "${INTERSHEET_REFS}" (id 0) (at 258.2715 32.1786 0)
-      (effects (font (size 1.27 1.27)) (justify left) hide)
-    )
-  )
-  (global_label "DAT2" (shape bidirectional) (at 159.258 57.658 180) (fields_autoplaced)
-    (effects (font (size 1.27 1.27)) (justify right))
-    (property "Intersheet References" "${INTERSHEET_REFS}" (id 0) (at 152.3981 57.5786 0)
-      (effects (font (size 1.27 1.27)) (justify right) hide)
-    )
-  )
-  (global_label "SCL" (shape bidirectional) (at 247.396 57.658 0) (fields_autoplaced)
-    (effects (font (size 1.27 1.27)) (justify left))
-    (property "Intersheet References" "${INTERSHEET_REFS}" (id 0) (at 253.2278 57.5786 0)
+  (global_label "CLK1" (shape bidirectional) (at 246.634 32.258 0) (fields_autoplaced)
+    (effects (font (size 1.27 1.27)) (justify left))
+    (property "Intersheet References" "${INTERSHEET_REFS}" (id 0) (at 253.7358 32.1786 0)
+      (effects (font (size 1.27 1.27)) (justify left) hide)
+    )
+  )
+  (global_label "SCL" (shape bidirectional) (at 159.258 57.658 180) (fields_autoplaced)
+    (effects (font (size 1.27 1.27)) (justify right))
+    (property "Intersheet References" "${INTERSHEET_REFS}" (id 0) (at 153.4262 57.5786 0)
+      (effects (font (size 1.27 1.27)) (justify right) hide)
+    )
+  )
+  (global_label "DAT2" (shape bidirectional) (at 247.396 57.658 0) (fields_autoplaced)
+    (effects (font (size 1.27 1.27)) (justify left))
+    (property "Intersheet References" "${INTERSHEET_REFS}" (id 0) (at 254.2559 57.5786 0)
       (effects (font (size 1.27 1.27)) (justify left) hide)
     )
@@
     )
   )
-  (global_label "DAT3" (shape bidirectional) (at 245.872 26.924 0) (fields_autoplaced)
-    (effects (font (size 1.27 1.27)) (justify left))
-    (property "Intersheet References" "${INTERSHEET_REFS}" (id 0) (at 252.7319 26.8446 0)
+  (global_label "CLK3" (shape bidirectional) (at 245.872 26.924 0) (fields_autoplaced)
+    (effects (font (size 1.27 1.27)) (justify left))
+    (property "Intersheet References" "${INTERSHEET_REFS}" (id 0) (at 252.9738 26.8446 0)
       (effects (font (size 1.27 1.27)) (justify left) hide)
     )
@@
     )
   )
-  (global_label "DS18b20" (shape bidirectional) (at 247.396 50.038 0) (fields_autoplaced)
-    (effects (font (size 1.27 1.27)) (justify left))
-    (property "Intersheet References" "${INTERSHEET_REFS}" (id 0) (at 258.1869 49.9586 0)
-      (effects (font (size 1.27 1.27)) (justify left) hide)
+  (global_label "DS18b20" (shape bidirectional) (at 159.512 62.738 180) (fields_autoplaced)
+    (effects (font (size 1.27 1.27)) (justify right))
+    (property "Intersheet References" "${INTERSHEET_REFS}" (id 0) (at 148.7211 62.6586 0)
+      (effects (font (size 1.27 1.27)) (justify right) hide)
     )
   )
@@
     )
   )
-  (global_label "DAT1" (shape bidirectional) (at 159.258 55.118 180) (fields_autoplaced)
-    (effects (font (size 1.27 1.27)) (justify right))
-    (property "Intersheet References" "${INTERSHEET_REFS}" (id 0) (at 152.3981 55.0386 0)
+  (global_label "SDA" (shape bidirectional) (at 159.258 55.118 180) (fields_autoplaced)
+    (effects (font (size 1.27 1.27)) (justify right))
+    (property "Intersheet References" "${INTERSHEET_REFS}" (id 0) (at 153.3657 55.0386 0)
       (effects (font (size 1.27 1.27)) (justify right) hide)
     )
@@
     )
   )
-  (global_label "CLK4" (shape bidirectional) (at 159.004 29.718 180) (fields_autoplaced)
-    (effects (font (size 1.27 1.27)) (justify right))
-    (property "Intersheet References" "${INTERSHEET_REFS}" (id 0) (at 151.9022 29.6386 0)
-      (effects (font (size 1.27 1.27)) (justify right) hide)
-    )
+  (global_label "Start_GPS" (shape output) (at 159.004 29.718 180) (fields_autoplaced)
+    (effects (font (size 1.27 1.27)) (justify right))
+    (property "Intersheet References" "${INTERSHEET_REFS}" (id 0) (at 147.3665 29.6386 0)
+      (effects (font (size 1.27 1.27)) (justify right) hide)
+    )
