File: untitled.kicad_sch (KiCad schematic)
At the start: 62 parts, among them IC5 HX711, IC6 HX711, IC7 HX711, IC8 HX711, J10 Conn_01x04, J15 Conn_01x04, J16 Conn_01x04, J2 Conn_01x04, J6 Conn_01x02, J7 Conn_01x02, Q2 MMBT4403, Q3 MMBT4403, Q4 MMBT4403, Q5 MMBT4403

Commit message: Update
Other:
- company: (none) -> Ratamuse
- title: (none) -> Open_beehive_scale_board
Changed lines of the file:
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@@
 (kicad_sch (version 20211123) (generator eeschema)
   (paper "A4")
+  (title_block
+    (title "Open_beehive_scale_board")
+    (date "2023-01-13")
+    (rev "V0.4")
+    (company "Ratamuse")
+  )
   (junction (at 30.48 34.29) (diameter 0) (color 0 0 0 0)
   )
